File: esp32_temperature_controller.kicad_sch (KiCad schematic)
At the start: 39 parts, among them J1 ESP32-DevKitC J1, J2 ESP32-DevKitC J2, J3 AC 220V, J4 Heater, J5 RTD1, J6 RTD2, J7 DHT20, U1 MAX31865xTP, U2 MAX31865xTP, U3 EL817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

Commit message: add debug port; change max31865 to ssop-20
Parts:
- added J8: JTAG, Connector_PinHeader_2.54mm:PinHeader_1x09_P2.54mm_Vertical, symbol Connector_Generic:Conn_01x09
- U1, U2: value MAX31865xTP -> MAX31865xAP; footprint Package_DFN_QFN:QFN-20-1EP_5x5mm_P0.65mm_EP3.35x3.35mm -> Package_SO:SSOP-20_5.3x7.2mm_P0.65mm; symbol Sensor_Temperature:MAX31865xTP -> Sensor_Temperature:MAX31865xAP
Connections:
- net +3V3: now also U1.2 (DVDD), U1.3 (VDD), U2.2 (DVDD), U2.3 (VDD); no longer U1.19 (DVDD), U1.20 (VDD), U2.19 (DVDD), U2.20 (VDD)
- net DHT_SCL: now also J1.17 (Pin_17); no longer J2.14 (Pin_14)
- net DHT_SDA: now also J1.16 (Pin_16); no longer J2.15 (Pin_15)
- net GND: now also U1.13 (GND), U1.18 (DGND), U1.19 (GND), U1.9 (FORCE2), U2.13 (GND), U2.18 (DGND), U2.19 (GND), U2.9 (FORCE2), J8.9 (Pin_9); no longer U1.10 (GND), U1.15 (DGND), U1.16 (GND), U1.21 (GND), U1.6 (FORCE2), U2.10 (GND), U2.15 (DGND), U2.16 (GND), U2.21 (GND), U2.6 (FORCE2)
- net HEATER_CTRL: now also J2.19 (Pin_19); no longer J1.18 (Pin_18)
- net TEMP1_CS: now also J1.6 (Pin_6), U1.16 (~{CS}); no longer J2.5 (Pin_5), U1.13 (~{CS})
- net TEMP1_RDY: now also J1.4 (Pin_4), U1.1 (~{DRDY}); no longer J2.3 (Pin_3), U1.18 (~{DRDY})
- net TEMP2_CS: now also J1.9 (Pin_9), U2.16 (~{CS}); no longer J2.10 (Pin_10), U2.13 (~{CS})
- net TEMP2_RDY: now also J1.10 (Pin_10), U2.1 (~{DRDY}); no longer J2.12 (Pin_12), U2.18 (~{DRDY})
- net TEMP_CLK: now also U1.15 (SCLK), U2.15 (SCLK); no longer U1.12 (SCLK), U2.12 (SCLK)
- net TEMP_DI: now also J1.7 (Pin_7), U1.14 (SDI), U2.14 (SDI); no longer J2.4 (Pin_4), U1.11 (SDI), U2.11 (SDI)
- net TEMP_DO: now also J1.8 (Pin_8), U1.17 (SDO), U2.17 (SDO); no longer J2.8 (Pin_8), U1.14 (SDO), U2.14 (SDO)
- net ZERO_CROSS: now also J2.18 (Pin_18); no longer J1.17 (Pin_17)
- net at C5.1, J5.3 (Pin_3): now also U1.11 (RTDIN-); no longer U1.8 (RTDIN-)
- net at C5.2, J5.2 (Pin_2): now also U1.10 (RTDIN+); no longer U1.7 (RTDIN+)
- net at J5.1 (Pin_1): now also U1.8 (FORCE+); no longer U1.5 (FORCE+)
- net at J5.4 (Pin_4): now also U1.12 (FORCE-); no longer U1.9 (FORCE-)
- net at J2.6 (Pin_6): no longer R9.2
- net at J6.1 (Pin_1): now also U2.8 (FORCE+); no longer U2.5 (FORCE+)
- net at C8.2, J6.2 (Pin_2): now also U2.10 (RTDIN+); no longer U2.7 (RTDIN+)
- net at C8.1, J6.3 (Pin_3): now also U2.11 (RTDIN-); no longer U2.8 (RTDIN-)
- net at J6.4 (Pin_4): now also U2.12 (FORCE-); no longer U2.9 (FORCE-)
- net MTDO: now reaches J2.16 (Pin_16)
- net MTDO: now also J8.4 (Pin_4)
- net MTMS: now reaches J1.12 (Pin_12)
- net MTMS: now also J8.3 (Pin_3)
- net MTDI: now reaches J1.13 (Pin_13)
- net MTDI: now also J8.1 (Pin_1)
- net MTCK: now reaches J1.15 (Pin_15)
- net MTCK: now also J8.2 (Pin_2)
- net EN: now reaches J1.2 (Pin_2)
- net EN: now also J8.5 (Pin_5)
- net LED_HEATER: now reaches J1.3 (Pin_3)
- net LED_HEATER: now also R10.1
- net at J1.5 (Pin_5): now also R9.2
- net LED_HEATING_STATE: no longer names the net of J2.2 (Pin_2)
- net LED_HEATING_STATE: no longer R10.1
- new net: R7.2, U1.4 (BIAS), U1.5 (REFIN+)
- new net: R7.1, U1.6 (REFIN-), U1.7 (ISENSOR)
- new net: R8.2, U2.4 (BIAS), U2.5 (REFIN+)
- new net: R8.1, U2.6 (REFIN-), U2.7 (ISENSOR)
- new net BOOT: J2.14 (Pin_14), J8.6 (Pin_6)
- new net RX0: J2.5 (Pin_5), J8.8 (Pin_8)
- new net TX0: J2.4 (Pin_4), J8.7 (Pin_7)
- no-connect marks 22 -> 14
Other:
- moved on the sheet: J1, J2, J7
